Commit message: xacro introduction

File: my_robot_description/urdf/my_robot.urdf.xacro (robot description, xacro)
@@ -1,4 +1,5 @@
 <?xml version="1.0"?>
-<robot name="my_robot">
+<robot name="my_robot" xmlns:xacro="http://www.ros.org/wiki/xacro">
+    <xacro:property name="base_length" value = "0.6"/>
     <material name="green">
         <color rgba="0 0.5 0 1"/>
@@ -11,5 +12,5 @@
         <visual>
             <geometry>
-                <box size="0.6 0.4 0.2"/>
+                <box size="${base_length} 0.4 0.2"/>
             </geometry>
             <origin xyz="0 0 0.1" rpy="0 0 0"/>
@@ -22,5 +23,5 @@
                 <cylinder radius="0.1" length="0.05"/>
             </geometry>
-            <origin xyz="0 0 0" rpy="1.57 0 0"/>
+            <origin xyz="0 0 0" rpy="${pi/2.0} 0 0"/>
             <material name="grey"/>
         </visual>
@@ -31,5 +32,5 @@
                 <cylinder radius="0.1" length="0.05"/>
             </geometry>
-            <origin xyz="0 0 0" rpy="1.57 0 0"/>
+            <origin xyz="0 0 0" rpy="${pi/2.0} 0 0"/>
             <material name="grey"/>
         </visual>
@@ -52,5 +53,5 @@
         <parent link="base_link"/>
         <child link="right_wheel_link"/>
-        <origin xyz = "-0.15 -0.225 0" rpy = "0 0 0"/>
+        <origin xyz = "${-base_length/4.0} -0.225 0" rpy = "0 0 0"/>
         <axis xyz = "0 1 0"/>
     </joint>
@@ -58,5 +59,5 @@
         <parent link="base_link"/>
         <child link="left_wheel_link"/>
-        <origin xyz = "-0.15 0.225 0" rpy = "0 0 0"/>
+        <origin xyz = "${-base_length/4.0} 0.225 0" rpy = "0 0 0"/>
         <axis xyz = "0 1 0"/>
     </joint>
@@ -64,5 +65,5 @@
         <parent link = "base_link"/>
         <child link = "caster_wheel_link"/>
-        <origin xyz = "0.2 0 -0.05" rpy = "0 0 0"/>
+        <origin xyz = "${base_length/3.0}  0 -0.05" rpy = "0 0 0"/>
     </joint>
 </robot>
